Commit message: Se agregan simulacion de gemelo digital mediante vectores de posicion por CLI

File: codigo/ros/src/Descripcion_Brazo/urdf/Brazo.urdf (robot description, URDF)
Before this commit: robot robot_master, 7 links, 6 joints
Joints:
- removed joint joint_base_to_hombro
- removed joint joint_eslabon_1_to_2
- removed joint joint_eslabon_2_to_3
- removed joint joint_eslabon_3_to_herramienta
- removed joint joint_hombro_to_eslabon_1
- added joint Servomotor 1: type revolute, parent base, child hombro_pitch, origin xyz=0 0 0.08 rpy=0 0 0, axis 0 0 1, limit lower=-3.14159 upper=3.14159 effort=10.0 velocity=1.0
- added joint Servomotor 2: type revolute, parent hombro_pitch, child eslabon_1, origin xyz=0 0 0 rpy=0 0 0, axis 0 1 0, limit lower=-3.14159 upper=3.14159 effort=10.0 velocity=1.0
- added joint Servomotor 3: type revolute, parent eslabon_1, child eslabon_2, origin xyz=0 0 0.10 rpy=0 0 0, axis 0 1 0, limit lower=-3.14159 upper=3.14159 effort=10.0 velocity=1.0
- added joint Servomotor 4: type revolute, parent eslabon_2, child eslabon_3, origin xyz=0 0 0.106 rpy=0 0 0, axis 0 1 0, limit lower=-3.14159 upper=3.14159 effort=10.0 velocity=1.0
- added joint Sin Servomotor: type fixed, parent eslabon_3, child herramienta, origin xyz=0.00101011 0 0.254243 rpy=0 -1.5708 0, axis 1 0 0, limit lower=-3.14159 upper=3.14159 effort=10.0 velocity=1.0
